File: pcb/business-card-synth.kicad_sch (KiCad schematic)
At the start: 79 parts, among them J1 Molex 48037-2200, J2 Conn_ARM_JTAG_SWD_10, J3 AudioJack4_SwitchTR1TR2, SW1 SW_SPDT, SW10 SW_Push, SW11 SW_Push, SW12 SW_Push, SW13 SW_Push, SW14 SW_Push, SW15 SW_Push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

Commit message: minor schematic updates. no pcb changes, no new revision
Other:
- note added: "Audio Output"
- note added: "Core"
- note added: "Keyboard"
- note added: "Power Supply"
- moved on the sheet: BT1, BT2, C1, C10, C11, C12, C13, C14, C15, C16, C17, C18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
