File: pcb/business-card-synth.kicad_sch (KiCad schematic)
At the start: 75 parts, among them J1 FTSH-105-01-L-DV-K, J2 Molex 48037-2200, J3 SJ1-3515-SMT-TR, Q1 2N7002, SW1 Wurth 450406020024, SW10 FSMSM, SW11 FSMSM, SW12 FSMSM, SW13 FSMSM, SW14 FSMSM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

Commit message: pcb: fix decoupling capacitors
100n capacitor must be closer to the supply pins.

no changes to fabrication layers, no new pcb revision.
Parts:
- renumbered C7 to C3, C3 to C7
Other:
- moved on the sheet: C3, C7
Changed lines of the file:
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@@
 	(symbol
 		(lib_id "Device:C_Small")
-		(at 142.24 62.23 180)
+		(at 101.6 62.23 180)
 		(unit 1)
 		(exclude_from_sim no)
@@
 		(dnp no)
 		(fields_autoplaced yes)
-		(property "Reference" "C7"
-			(at 144.78 60.9535 0)
+		(property "Reference" "C3"
+			(at 104.14 60.9535 0)
 			(effects
 				(font
@@
 		)
 		(property "Value" "100n"
-			(at 144.78 63.4935 0)
+			(at 104.14 63.4935 0)
 			(effects
 				(font
@@
 		)
 		(property "Footprint" "Capacitor_SMD:C_0805_2012Metric"
-			(at 142.24 62.23 0)
+			(at 101.6 62.23 0)
 			(effects
 				(font
@@
 		)
 		(property "Datasheet" "~"
-			(at 142.24 62.23 0)
+			(at 101.6 62.23 0)
 			(effects
 				(font
@@
 		)
 		(property "Description" "Unpolarized capacitor, small symbol"
-			(at 142.24 62.23 0)
+			(at 101.6 62.23 0)
 			(effects
 				(font
@@
 		)
 		(property "Mouser No." "603-CC805KRX7R9BB104"
-			(at 142.24 62.23 0)
+			(at 101.6 62.23 0)
 			(effects
 				(font
@@
 			(project "business-card-synth"
 				(path "/ecb6e53c-6b1b-4bf5-a63a-cd7c5ac0c026"
-					(reference "C7")
+					(reference "C3")
 					(unit 1)
 				)
@@
 	(symbol
 		(lib_id "Device:C_Small")
-		(at 101.6 62.23 180)
+		(at 142.24 62.23 180)
 		(unit 1)
 		(exclude_from_sim no)
@@
 		(dnp no)
 		(fields_autoplaced yes)
-		(property "Reference" "C3"
-			(at 104.14 60.9535 0)
+		(property "Reference" "C7"
+			(at 144.78 60.9535 0)
 			(effects
 				(font
@@
 		)
 		(property "Value" "10u"
-			(at 104.14 63.4935 0)
+			(at 144.78 63.4935 0)
 			(effects
 				(font
@@
 		)
 		(property "Footprint" "Capacitor_SMD:C_0805_2012Metric"
-			(at 101.6 62.23 0)
+			(at 142.24 62.23 0)
 			(effects
 				(font
@@
 		)
 		(property "Datasheet" "~"
-			(at 101.6 62.23 0)
+			(at 142.24 62.23 0)
 			(effects
 				(font
@@
 		)
 		(property "Description" "Unpolarized capacitor, small symbol"
-			(at 101.6 62.23 0)
+			(at 142.24 62.23 0)
 			(effects
 				(font
@@
 		)
 		(property "Mouser No." "603-CC805KKX7R6BB106"
-			(at 101.6 62.23 0)
+			(at 142.24 62.23 0)
 			(effects
 				(font
@@
 			(project "business-card-synth"
 				(path "/ecb6e53c-6b1b-4bf5-a63a-cd7c5ac0c026"
-					(reference "C3")
+					(reference "C7")
 					(unit 1)
 				)
