File: pcb/business-card-synth.kicad_pcb (KiCad board)
At the start: 2 copper layers, 85.6 x 78.4 mm, 90 parts, among them J1 FTSH-105-01-L-DV-K, J2 Molex 48037-2200, J3 SJ1-3515-SMT-TR, Q1 2N7002, SW1 Wurth 450406020024, SW10 FSMSM, SW11 FSMSM, SW12 FSMSM, SW13 FSMSM, SW14 FSMSM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

Commit message: pcb: fix decoupling capacitors
100n capacitor must be closer to the supply pins.

no changes to fabrication layers, no new pcb revision.
Parts:
- C3: value 10u -> 100n
- C7: value 100n -> 10u
Changed lines of the file:
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@@
 			)
 		)
-		(property "Value" "10u"
+		(property "Value" "100n"
 			(at 0 -1.68 90)
 			(layer "B.Fab")
@@
 			)
 		)
-		(property "Mouser No." "603-CC805KKX7R6BB106"
+		(property "Mouser No." "603-CC805KRX7R9BB104"
 			(at 0 0 270)
 			(unlocked yes)
@@
 			)
 		)
-		(property "Value" "100n"
+		(property "Value" "10u"
 			(at 0 -1.68 90)
 			(layer "B.Fab")
@@
 			)
 		)
-		(property "Mouser No." "603-CC805KRX7R9BB104"
+		(property "Mouser No." "603-CC805KKX7R6BB106"
 			(at 0 0 270)
 			(unlocked yes)
